File: hardware/CarTalk.brd (EAGLE design)
At the start: 38.1 x 40.6 mm, 42 parts, among them J4 1X10, J5 1X10

Commit message: Renamed files to match project name
Parts:
- C1, C11, C12, C13, C14, C16, C2, C3, C4, C5, C6, C7, C9: device CarTalkImu:C0603 -> CarTalk:C0603
- C10, C15, C8: device CarTalkImu:C0805 -> CarTalk:C0805
- FB1, R1, R10, R11, R12, R2, R3, R4, R5, R6, R7, R8, R9: device CarTalkImu:R0603 -> CarTalk:R0603
- GPS: device CarTalkImu:CAM-M8 -> CarTalk:CAM-M8
- J4, J5: device CarTalkImu:1X10 -> CarTalk:1X10
- MPU: device CarTalkImu:QFN24-NP -> CarTalk:QFN24-NP
- TPH: device CarTalkImu:BME-DFN8 -> CarTalk:BME-DFN8
- U$10, U$11, U$6, U$7, U$8, U$9: device CarTalkImu:FIDUCIAL_1MM -> CarTalk:FIDUCIAL_1MM
- U$5: device CarTalkImu:SILK_QC -> CarTalk:SILK_QC
- WIFI: device CarTalkImu:ESP-12 -> CarTalk:ESP-12
